File: v_0.1/hardware/gpswidget/gpswidget.sch (KiCad schematic (older format))
At the start: 13 parts

Commit message: update
Parts:
- added J?: Conn_01x04_Female, symbol Connector:Conn_01x04_Female
- added JP?: Jumper_NO_Small, symbol Device:Jumper_NO_Small
- added R? (x2): R, symbol Device:R
- U2: renamed from U?; footprint (none) -> footprints:RFM95
- gave numbers to parts that had none: 12
Connections:
- net +3V3: now also JP?.1, R?.1, R?.1
- net 3V_SWITCH: now also J?.2 (Pin_2), JP?.2
- net GND: now also J?.1 (Pin_1)
- net 16 renamed SCL
- net SCL: now also J?.3 (Pin_3), R?.2
- net 17 renamed SDA
- net SDA: now also J?.4 (Pin_4), R?.2
Other:
- note added: "LDO"
- note added: "i2c pullups"
- note added: "oled"
Changed lines of the file:
@@
 $EndDescr
 $Comp
-L MCU_Microchip_ATmega:ATmega1284P-PU U?
+L MCU_Microchip_ATmega:ATmega1284P-PU U1
 U 1 1 6061E5F3
 P 2850 3150
-F 0 "U?" H 2000 2300 50  0000 C CNN
+F 0 "U1" H 2000 2300 50  0000 C CNN
 F 1 "ATmega1284P-PU" H 1950 2150 50  0000 C CNN
 F 2 "Package_DIP:DIP-40_W15.24mm" H 2850 3150 50  0001 C CIN
@@
 $EndComp
 $Comp
-L Connector:Conn_01x04_Female J?
+L Connector:Conn_01x04_Female J2
 U 1 1 6061F728
 P 4900 1100
-F 0 "J?" H 4928 1076 50  0000 L CNN
+F 0 "J2" H 4928 1076 50  0000 L CNN
 F 1 "Conn_01x04_Female" H 4928 985 50  0000 L CNN
 F 2 "" H 4900 1100 50  0001 C CNN
@@
 GPS
 $Comp
-L RF_Module:RFM95W-915S2 U?
+L RF_Module:RFM95W-915S2 U2
 U 1 1 606219F2
 P 6850 1450
-F 0 "U?" H 6850 2131 50  0000 C CNN
+F 0 "U2" H 6850 2131 50  0000 C CNN
 F 1 "RFM95W-915S2" H 6850 2040 50  0000 C CNN
-F 2 "" H 3550 3100 50  0001 C CNN
+F 2 "footprints:RFM95" H 3550 3100 50  0001 C CNN
 F 3 "https://www.hoperf.com/data/upload/portal/20181127/5bfcbea20e9ef.pdf" H 3550 3100 50  0001 C CNN
 	1    6850 1450
@@
 $EndComp
 $Comp
-L Connector:Conn_01x12_Female J?
+L Connector:Conn_01x12_Female J1
 U 1 1 606248C2
 P 4800 2550
-F 0 "J?" H 4828 2526 50  0000 L CNN
+F 0 "J1" H 4828 2526 50  0000 L CNN
 F 1 "Conn_01x12_Female" H 4828 2435 50  0000 L CNN
 F 2 "" H 4800 2550 50  0001 C CNN
@@
 eink breakout
 $Comp
-L Connector:Micro_SD_Card J?
+L Connector:Micro_SD_Card J3
 U 1 1 60621969
 P 9550 1450
-F 0 "J?" H 9500 2167 50  0000 C CNN
+F 0 "J3" H 9500 2167 50  0000 C CNN
 F 1 "Micro_SD_Card" H 9500 2076 50  0000 C CNN
 F 2 "" H 10700 1750 50  0001 C CNN
@@
 $EndComp
 $Comp
-L Device:LED D?
+L Device:LED D1
 U 1 1 606350FC
 P 6300 3200
-F 0 "D?" V 6339 3083 50  0000 R CNN
+F 0 "D1" V 6339 3083 50  0000 R CNN
 F 1 "LED" V 6248 3083 50  0000 R CNN
 F 2 "" H 6300 3200 50  0001 C CNN
@@
 $EndComp
 $Comp
-L Device:R R?
+L Device:R R2
 U 1 1 60635D60
 P 6300 2900
-F 0 "R?" H 6370 2946 50  0000 L CNN
+F 0 "R2" H 6370 2946 50  0000 L CNN
 F 1 "R" H 6370 2855 50  0000 L CNN
 F 2 "" V 6230 2900 50  0001 C CNN
@@
 	6300 2750 6300 2600
 $Comp
-L power:GND #PWR?
+L power:GND #PWR0101
 U 1 1 60639DB7
 P 6300 3350
-F 0 "#PWR?" H 6300 3100 50  0001 C CNN
+F 0 "#PWR0101" H 6300 3100 50  0001 C CNN
 F 1 "GND" H 6305 3177 50  0000 C CNN
 F 2 "" H 6300 3350 50  0001 C CNN
@@
 4
 $Comp
-L power:GND #PWR?
+L power:GND #PWR0102
 U 1 1 60649079
 P 4700 1000
-F 0 "#PWR?" H 4700 750 50  0001 C CNN
+F 0 "#PWR0102" H 4700 750 50  0001 C CNN
 F 1 "GND" V 4705 872 50  0000 R CNN
 F 2 "" H 4700 1000 50  0001 C CNN
@@
 3V_SWITCH
 $Comp
-L power:GND #PWR?
+L power:GND #PWR0103
 U 1 1 60651931
 P 8250 1650
-F 0 "#PWR?" H 8250 1400 50  0001 C CNN
+F 0 "#PWR0103" H 8250 1400 50  0001 C CNN
 F 1 "GND" H 8255 1477 50  0000 C CNN
 F 2 "" H 8250 1650 50  0001 C CNN
@@
 MOSI
 $Comp
-L power:GND #PWR?
+L power:GND #PWR0104
 U 1 1 606533A5
 P 10350 2050
-F 0 "#PWR?" H 10350 1800 50  0001 C CNN
+F 0 "#PWR0104" H 10350 1800 50  0001 C CNN
 F 1 "GND" H 10355 1877 50  0000 C CNN
 F 2 "" H 10350 2050 50  0001 C CNN
@@
 $EndComp
 $Comp
-L power:GND #PWR?
+L power:GND #PWR0105
 U 1 1 6065D5EE
 P 4600 2250
-F 0 "#PWR?" H 4600 2000 50  0001 C CNN
+F 0 "#PWR0105" H 4600 2000 50  0001 C CNN
 F 1 "GND" V 4605 2122 50  0000 R CNN
 F 2 "" H 4600 2250 50  0001 C CNN
@@
 $EndComp
 $Comp
-L power:+3V3 #PWR?
+L power:+3V3 #PWR0106
 U 1 1 6065E09E
 P 4600 2050
-F 0 "#PWR?" H 4600 1900 50  0001 C CNN
+F 0 "#PWR0106" H 4600 1900 50  0001 C CNN
 F 1 "+3V3" H 4615 2223 50  0000 C CNN
 F 2 "" H 4600 2050 50  0001 C CNN
@@
 SCK
 $Comp
-L power:GND #PWR?
+L power:GND #PWR0107
 U 1 1 60665EE6
 P 6750 2050
-F 0 "#PWR?" H 6750 1800 50  0001 C CNN
+F 0 "#PWR0107" H 6750 1800 50  0001 C CNN
 F 1 "GND" H 6755 1877 50  0000 C CNN
 F 2 "" H 6750 2050 50  0001 C CNN
@@
 7
 Text GLabel 3450 3250 2    50   Input ~ 0
-16
+SCL
 Text GLabel 3450 3350 2    50   Input ~ 0
-17
+SDA
 Text GLabel 3450 3450 2    50   Input ~ 0
 18
@@
 15
 $Comp
-L power:GND #PWR?
+L power:GND #PWR0108
 U 1 1 6068DD1E
 P 2850 5150
-F 0 "#PWR?" H 2850 4900 50  0001 C CNN
+F 0 "#PWR0108" H 2850 4900 50  0001 C CNN
 F 1 "GND" H 2855 4977 50  0000 C CNN
 F 2 "" H 2850 5150 50  0001 C CNN
@@
 $EndComp
 $Comp
-L Device:C C?
+L Device:C C4
 U 1 1 60690C3F
 P 1950 2450
-F 0 "C?" H 2065 2496 50  0000 L CNN
+F 0 "C4" H 2065 2496 50  0000 L CNN
 F 1 "0.1uF" H 2065 2405 50  0000 L CNN
 F 2 "" H 1988 2300 50  0001 C CNN
@@
 $EndComp
 $Comp
-L power:GND #PWR?
+L power:GND #PWR0109
 U 1 1 60691979
 P 1950 2600
-F 0 "#PWR?" H 1950 2350 50  0001 C CNN
+F 0 "#PWR0109" H 1950 2350 50  0001 C CNN
 F 1 "GND" H 1955 2427 50  0000 C CNN
 F 2 "" H 1950 2600 50  0001 C CNN
@@
 	2950 1150 2850 1150
 $Comp
-L power:+3V3 #PWR?
+L power:+3V3 #PWR0110
 U 1 1 60694BA9
 P 2850 900
-F 0 "#PWR?" H 2850 750 50  0001 C CNN
+F 0 "#PWR0110" H 2850 750 50  0001 C CNN
 F 1 "+3V3" H 2865 1073 50  0000 C CNN
 F 2 "" H 2850 900 50  0001 C CNN
@@
 	1950 1450 1950 1250
 $Comp
-L Device:R R?
+L Device:R R1
 U 1 1 606A07E7
 P 1950 1100
-F 0 "R?" H 2020 1146 50  0000 L CNN
+F 0 "R1" H 2020 1146 50  0000 L CNN
 F 1 "10K" H 2020 1055 50  0000 L CNN
 F 2 "" V 1880 1100 50  0001 C CNN
@@
 Connection ~ 1950 1450
 $Comp
-L Device:C C?
+L Device:C C1
 U 1 1 606A2D75
 P 900 1600
-F 0 "C?" H 1015 1646 50  0000 L CNN
+F 0 "C1" H 1015 1646 50  0000 L CNN
 F 1 "0.1uF" H 1015 1555 50  0000 L CNN
 F 2 "" H 938 1450 50  0001 C CNN
@@
 DTR
 $Comp
-L Device:Crystal Y?
+L Device:Crystal Y1
 U 1 1 606A633A
 P 2050 1750
-F 0 "Y?" V 2004 1881 50  0000 L CNN
+F 0 "Y1" V 2004 1881 50  0000 L CNN
 F 1 "Crystal" V 2095 1881 50  0000 L CNN
 F 2 "" H 2050 1750 50  0001 C CNN
@@
 Connection ~ 2050 1900
 $Comp
-L Device:C C?
+L Device:C C2
 U 1 1 606AB90C
 P 1700 1600
-F 0 "C?" V 1650 1450 50  0000 C CNN
+F 0 "C2" V 1650 1450 50  0000 C CNN
 F 1 "22pF" V 1750 1450 50  0000 C CNN
 F 2 "" H 1738 1450 50  0001 C CNN
@@
 $EndComp
 $Comp
-L Device:C C?
+L Device:C C3
 U 1 1 606ABF72
 P 1700 1900
-F 0 "C?" V 1650 1700 50  0000 C CNN
+F 0 "C3" V 1650 1700 50  0000 C CNN
 F 1 "22pF" V 1750 1700 50  0000 C CNN
 F 2 "" H 1738 1750 50  0001 C CNN
@@
 Connection ~ 1350 1900
 $Comp
-L power:GND #PWR?
+L power:GND #PWR0111
 U 1 1 606B495A
 P 1350 2050
-F 0 "#PWR?" H 1350 1800 50  0001 C CNN
+F 0 "#PWR0111" H 1350 1800 50  0001 C CNN
 F 1 "GND" H 1355 1877 50  0000 C CNN
 F 2 "" H 1350 2050 50  0001 C CNN
@@
 Wire Wire Line
 	1950 2050 1950 2300
+Text Notes 4900 3850 0    50   ~ 0
+LDO
+$Comp
+L Connector:Conn_01x04_Female J?
+U 1 1 606F7027
+P 6100 5050
+F 0 "J?" H 6128 5026 50  0000 L CNN
+F 1 "Conn_01x04_Female" H 6128 4935 50  0000 L CNN
+F 2 "" H 6100 5050 50  0001 C CNN
+F 3 "~" H 6100 5050 50  0001 C CNN
+	1    6100 5050
+	1    0    0    -1
+$EndComp
+$Comp
+L power:GND #PWR?
+U 1 1 606F76DA
+P 5900 4950
+F 0 "#PWR?" H 5900 4700 50  0001 C CNN
+F 1 "GND" V 5905 4822 50  0000 R CNN
+F 2 "" H 5900 4950 50  0001 C CNN
+F 3 "" H 5900 4950 50  0001 C CNN
+	1    5900 4950
+	0    1    1    0
+$EndComp
+Text GLabel 5900 5150 0    50   Input ~ 0
+SCL
+Text GLabel 5900 5250 0    50   Input ~ 0
+SDA
+Text Notes 5850 4800 0    50   ~ 0
+oled
+$Comp
+L Device:R R?
+U 1 1 606FEBFC
+P 7300 5100
+F 0 "R?" H 7370 5146 50  0000 L CNN
+F 1 "R" H 7370 5055 50  0000 L CNN
+F 2 "" V 7230 5100 50  0001 C CNN
+F 3 "~" H 7300 5100 50  0001 C CNN
+	1    7300 5100
+	1    0    0    -1
+$EndComp
+Text GLabel 7300 5250 0    50   Input ~ 0
+SCL
+$Comp
+L power:+3V3 #PWR?
+U 1 1 606FFBBF
+P 7300 4950
+F 0 "#PWR?" H 7300 4800 50  0001 C CNN
+F 1 "+3V3" H 7315 5123 50  0000 C CNN
+F 2 "" H 7300 4950 50  0001 C CNN
+F 3 "" H 7300 4950 50  0001 C CNN
+	1    7300 4950
+	1    0    0    -1
+$EndComp
+$Comp
+L Device:R R?
+U 1 1 6070008A
+P 7700 5100
+F 0 "R?" H 7770 5146 50  0000 L CNN
+F 1 "R" H 7770 5055 50  0000 L CNN
+F 2 "" V 7630 5100 50  0001 C CNN
+F 3 "~" H 7700 5100 50  0001 C CNN
+	1    7700 5100
+	1    0    0    -1
+$EndComp
+Text GLabel 7700 5250 0    50   Input ~ 0
+SDA
+$Comp
+L power:+3V3 #PWR?
+U 1 1 6070042D
+P 7700 4950
+F 0 "#PWR?" H 7700 4800 50  0001 C CNN
+F 1 "+3V3" H 7715 5123 50  0000 C CNN
+F 2 "" H 7700 4950 50  0001 C CNN
+F 3 "" H 7700 4950 50  0001 C CNN
+	1    7700 4950
+	1    0    0    -1
+$EndComp
+Text Notes 7400 4650 0    50   ~ 0
+i2c pullups
+$Comp
+L power:+3V3 #PWR?
+U 1 1 606F8952
+P 4950 4850
+F 0 "#PWR?" H 4950 4700 50  0001 C CNN
+F 1 "+3V3" H 4965 5023 50  0000 C CNN
+F 2 "" H 4950 4850 50  0001 C CNN
+F 3 "" H 4950 4850 50  0001 C CNN
+	1    4950 4850
+	1    0    0    -1
+$EndComp
+$Comp
+L Device:Jumper_NO_Small JP?
+U 1 1 6070F0B3
+P 5050 5050
+F 0 "JP?" H 5050 5235 50  0000 C CNN
+F 1 "Jumper_NO_Small" H 5050 5144 50  0000 C CNN
+F 2 "" H 5050 5050 50  0001 C CNN
+F 3 "~" H 5050 5050 50  0001 C CNN
+	1    5050 5050
+	1    0    0    -1
+$EndComp
+Wire Wire Line
+	4950 5050 4950 4850
+Wire Wire Line
+	5150 5050 5250 5050
+Text GLabel 5150 5300 0    50   Input ~ 0
+3V_SWITCH
+Wire Wire Line
+	5150 5300 5250 5300
+Wire Wire Line
+	5250 5300 5250 5050
+Connection ~ 5250 5050
+Wire Wire Line
+	5250 5050 5900 5050
 $EndSCHEMATC
